Commit message: Take videos!

File: assets/urdf/cartpole2.urdf (robot description, URDF)
Before this commit: robot cartpole, 6 links, 5 joints
Joints:
- joint camera_mount_to_camera_tilt: limit lower=-1.57 upper=1.57 effort=0.1 velocity=0.01 -> lower=-1.57 upper=1.57 effort=1000 velocity=100
- joint cart_to_camera_pan: limit lower=-1.57 upper=1.57 effort=0.1 velocity=0.01 -> lower=-1.57 upper=1.57 effort=1000 velocity=100
- joint slider1_to_slider2: limit lower=0 upper=0 effort=1000.0 velocity=100 -> lower=-10 upper=10 effort=1000.0 velocity=100
- joint slider2_to_cart: limit lower=0 upper=0 effort=1000.0 velocity=100 -> lower=-10 upper=10 effort=1000.0 velocity=100
